File: PCB/mini keyboard 2.kicad_pcb (KiCad board)
At the start: 2 copper layers, 98.5 x 40.8 mm, 13 parts, among them SW1 SW_Push, SW2 SW_Push, SW3 SW_Push, SW4 SW_Push, SW5 SW_Push, SW6 SW_Push, SW7 SW_Push, SW8 SW_Push, SW9 RotaryEncoder_Switch, U1 XIAO-RP2040-DIP

Commit message: Update files
Parts:
- SW9: moved to F.Cu
- moved SW9 85.5 mm to (121.2, 51.6), turned to 0 degrees
- moved D3 78.5 mm to (128.2, 26.9), turned to 180 degrees
- moved D2 74.6 mm to (128.2, 31.6), turned to 180 degrees
- moved D1 71.7 mm to (128.2, 36.4), turned to 180 degrees
- moved SW3 71.4 mm to (72.9, 30.1)
- moved SW4 71.4 mm to (72.9, 49.2)
- moved SW1 71.4 mm to (53.8, 30.1)
- moved SW2 71.4 mm to (53.8, 49.2)
- moved SW5 71.4 mm to (91.9, 30.1)
- moved SW6 71.4 mm to (91.9, 49.2)
- moved SW7 71.4 mm to (111.0, 30.1)
- moved SW8 71.4 mm to (111.0, 49.2)
- moved U1 71.4 mm to (128.4, 34.9)
Routing:
- net Net-(D1-DIN): track 29.5 -> 14.0 mm
- net Net-(U1-GPIO27/ADC1/A1): track 23.1 -> 36.0 mm
- net Net-(U1-GPIO26/ADC0/A0): track 31.0 -> 41.5 mm
- net +5V: track 30.5 -> 22.2 mm
- net GND: track 263.4 -> 261.9 mm
Other:
- board size 98.5 x 40.8 mm -> 98.5 x 40.6 mm

Commit message: Update files
Parts:
- D1, D2, D3: moved to F.Cu
- moved D1 11.2 mm to (128.8, 25.1), turned to 0 degrees
- moved D3 7.84 mm to (128.8, 34.7), turned to 0 degrees
- moved D2 1.80 mm to (128.8, 29.9), turned to 0 degrees
Routing:
- net Net-(D1-DOUT): track 7.66 -> 15.6 mm, vias 0 -> 2
- net +5V: track 22.2 -> 30.1 mm
- net Net-(D2-DOUT): track 7.52 -> 15.1 mm, vias 0 -> 2
- net GND: track 261.9 -> 258.1 mm
- net Net-(D1-DIN): track 14.0 -> 11.0 mm, vias 0 -> 1
